File: interface_us_board.brd (EAGLE design)
At the start: 160 x 107.8 mm, 38 parts, among them IC1 74AC245DW, IC2 4050D

Commit message: Revert "InterfaceUSBoard: change resistor value" change was not needed
This reverts commit 6388b83db6797b02bafabf1e9fd2be2e5c524c07.
Parts:
- R1: value 100 -> 47
Changed lines of the file:
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@@
 <attribute name="OC_FARNELL" value="unknown" x="-87.055" y="-29.005" size="1.778" layer="27" rot="R270" display="off"/>
 </element>
-<element name="R1" library="resistor" package="M1206" value="100" x="36.068" y="60.2996" rot="MR90"/>
+<element name="R1" library="resistor" package="M1206" value="47" x="36.068" y="60.2996" rot="MR90"/>
 <element name="IC1" library="74xx-eu" package="SO20W" value="74AC245DW" x="-27.195" y="-4.155" rot="R270"/>
 <element name="IC2" library="40xx" package="SO16" value="4050D" x="-55.74" y="-1.365" rot="R90"/>

Commit message: InterfaceUSBoard: change resistor value
Parts:
- R1: value 47 -> 100
Changed lines of the file:
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@@
 <attribute name="OC_FARNELL" value="unknown" x="-87.055" y="-29.005" size="1.778" layer="27" rot="R270" display="off"/>
 </element>
-<element name="R1" library="resistor" package="M1206" value="47" x="36.068" y="60.2996" rot="MR90"/>
+<element name="R1" library="resistor" package="M1206" value="100" x="36.068" y="60.2996" rot="MR90"/>
 <element name="IC1" library="74xx-eu" package="SO20W" value="74AC245DW" x="-27.195" y="-4.155" rot="R270"/>
 <element name="IC2" library="40xx" package="SO16" value="4050D" x="-55.74" y="-1.365" rot="R90"/>
