File: ec_motor_board.brd (EAGLE design)
At the start: 28 x 50 mm, 23 parts

Commit message: ec_motor_board: necessary pullups to 3.3v connected to hall sensors leiton.dru: added for drc with leiton values
Parts:
- added R10, R11, R12: (no value), resistor:R1206
- moved D1 1.66 mm to (17.8, 6.99)
- moved D2 1.66 mm to (17.8, 9.53)
- moved R4 1.66 mm to (11.5, 8.26)
- moved C5 1.47 mm to (13.9, 8.26)
- moved C8 1.47 mm to (21.7, 8.26)
- moved C9 1.47 mm to (24.0, 8.26)
Connections:
- net N$19: now also R10.1
- net N$21: now also R11.2
- net N$23: now also R12.2
- net VCC: now also R10.2, R11.1, R12.1
Routing:
- net N$23: track 35.3 -> 55.7 mm, vias 2 -> 6
- net N$21: track 28.8 -> 46.9 mm, vias 2 -> 6
- net N$19: track 34.3 -> 52.2 mm, vias 0 -> 2
- net VCC: track 0.00 -> 10.4 mm
- net N$4: track 18.0 -> 21.7 mm
- net N$9: track 25.7 -> 28.2 mm
- net N$12: track 31.2 -> 33.3 mm
- net N$6: track 38.2 -> 36.2 mm
- net N$8: track 62.7 -> 61.0 mm
- net GND: track 150.3 -> 150.9 mm
- net N$27: track 44.4 -> 45.0 mm

Commit message: ec_motor_board: added an 0 ohm resistor which can connect vref to vcc to disable power regulation
Parts:
- added R13: 0, resistor:R1206
- moved R12 0.65 mm to (6.83, 8.57)
- moved R4 0.32 mm to (11.8, 8.26)
- moved C5 0.16 mm to (14.0, 8.26)
Connections:
- net N$14: now also R13.2
- net VCC: now also R13.1
Routing:
- net VCC: track 10.4 -> 16.6 mm
- net N$14: track 22.1 -> 27.6 mm, vias 1 -> 2
- net GND: track 150.9 -> 150.0 mm
- net N$23: track 55.7 -> 56.6 mm
- net N$7: track 68.8 -> 69.4 mm
- net N$1: track 38.1 -> 37.5 mm
- net N$8: track 61.0 -> 61.6 mm
