File: tsop.sch (EAGLE design)
At the start: 193 parts, among them IC1 4051D, IC2 4051D, IC3 4051D, IC4 4051D, IC5 MEGA48/88/168-PU

Commit message: TSOP: set TSOPs to the right position and started to wire low pass filters
Parts:
- removed 22_24, 22_25, 22_26, 22_27, 22_28, 22_29, 22_30, 22_31: TSOP2240, ShortCircuitRobotics:TSOP2240
- removed C49, C51, C53, C55, C57, C59, C61, C63: 1µF, resistor:C-EUC1206
- removed C50, C52, C54, C56, C58, C60, C62, C64: 4.7µF, resistor:C-EUC1206
- removed IC4: 4051D, 40xx:4051D
- removed R49, R51, R53, R55, R57, R59, R61, R63: 100k, resistor:R-EU_M1206
- removed R50, R52, R54, R56, R58, R60, R62, R64: 100, resistor:R-EU_M1206
Connections:
- removed net MUX_INH_3: IC4A.INH, IC5.PD5(T1/OC0B/PCINT21)
- removed net N$49: 22_24.V+, C50.1, R50.1
- removed net N$50: 22_24.OUT, R49.1
- removed net N$51: 22_25.V+, C52.1, R52.1
- removed net N$52: 22_25.OUT, R51.1
- removed net N$53: 22_26.V+, C54.1, R54.1
- removed net N$54: 22_26.OUT, R53.1
- removed net N$55: 22_27.V+, C56.1, R56.1
- removed net N$56: 22_27.OUT, R55.1
- removed net N$57: 22_28.V+, C58.1, R58.1
- removed net N$58: 22_28.OUT, R57.1
- removed net N$59: 22_29.V+, C60.1, R60.1
- removed net N$60: 22_29.OUT, R59.1
- removed net N$61: 22_30.V+, C62.1, R62.1
- removed net N$62: 22_30.OUT, R61.1
- removed net N$63: 22_31.V+, C64.1, R64.1
- removed net N$64: 22_31.OUT, R63.1
- removed net TSOP24: C55.1, IC4A.X0, R55.2
- removed net TSOP25: C53.1, IC4A.X1, R53.2
- removed net TSOP26: C51.1, IC4A.X2, R51.2
- removed net TSOP27: C49.1, IC4A.X3, R49.2
- removed net TSOP28: C63.1, IC4A.X4, R63.2
- removed net TSOP29: C61.1, IC4A.X5, R61.2
- removed net TSOP30: C59.1, IC4A.X6, R59.2
- removed net TSOP31: C57.1, IC4A.X7, R57.2
- net GND: now also C66.2; no longer 22_24.GND, 22_25.GND, 22_26.GND, 22_27.GND, 22_28.GND, 22_29.GND, 22_30.GND, 22_31.GND, C49.2, C50.2, C51.2, C52.2, C53.2, C54.2, C55.2, C56.2, C57.2, C58.2, C59.2, C60.2, C61.2, C62.2, C63.2, C64.2
- net MUX_A: no longer IC4A.A
- net MUX_B: no longer IC4A.B
- net MUX_C: no longer IC4A.C
- net MUX_OUT: no longer IC4A.X
- net N$81: now also IC5.PB7(XTAL2/TOSC2/PCINT7)
- net VCC: no longer C66.2
- net VTSOP_A: no longer R50.2, R58.2
- net VTSOP_B: no longer R52.2, R60.2
- net VTSOP_C: no longer R54.2, R62.2
- net VTSOP_D: no longer R56.2, R64.2
Other:
- moved on the sheet: C66

Commit message: TSOP: finished TSOP.sch and TSOP.brd 	TSOP data wires were connected with wrong TSOPS
Connections:
- net GND: now also IC1P.GND, IC1P.VEE, IC2P.GND, IC2P.VEE, IC3P.GND, IC3P.VEE
- net TSOP0: now also C28.1, R13.2; no longer C6.1, R6.2
- net TSOP1: now also C1.1, R2.2; no longer C3.1, R4.2
- net TSOP10: now also C20.1, R21.2; no longer C18.1, R19.2
- net TSOP11: now also C22.1, R23.2; no longer C16.1, R17.2
- net TSOP12: now also C24.1, R25.2; no longer C31.1, R31.2
- net TSOP13: now also C26.1, R27.2; no longer C29.1, R29.2
- net TSOP14: now also C29.1, R29.2; no longer C26.1, R27.2
- net TSOP15: now also C31.1, R31.2; no longer C24.1, R25.2
- net TSOP16: now also C33.1, R33.2; no longer C39.1, R39.2
- net TSOP17: now also C35.1, R35.2; no longer C37.1, R37.2
- net TSOP18: now also C37.1, R37.2; no longer C35.1, R35.2
- net TSOP19: now also C39.1, R39.2; no longer C33.1, R33.2
- net TSOP2: now also C3.1, R4.2; no longer C1.1, R2.2
- net TSOP20: now also C41.1, R41.2; no longer C47.1, R47.2
- net TSOP21: now also C43.1, R43.2; no longer C45.1, R45.2
- net TSOP22: now also C45.1, R45.2; no longer C43.1, R43.2
- net TSOP23: now also C47.1, R47.2; no longer C41.1, R41.2
- net TSOP3: now also C6.1, R6.2; no longer C28.1, R13.2
- net TSOP4: now also C8.1, R8.2; no longer C14.1, R15.2
- net TSOP5: now also C10.1, R10.2; no longer C12.1, R12.2
- net TSOP6: now also C12.1, R12.2; no longer C10.1, R10.2
- net TSOP7: now also C14.1, R15.2; no longer C8.1, R8.2
- net TSOP8: now also C16.1, R17.2; no longer C22.1, R23.2
- net TSOP9: now also C18.1, R19.2; no longer C20.1, R21.2
- net VCC: now also IC1P.VCC, IC2P.VCC, IC3P.VCC
