File: tsop.brd (EAGLE design)
At the start: 100 x 80 mm, 193 parts, among them IC1 4051D, IC2 4051D, IC3 4051D, IC4 4051D, IC5 MEGA48/88/168-PU

Commit message: TSOP: set TSOPs to the right position and started to wire low pass filters
Parts:
- removed 22_24, 22_25, 22_26, 22_27, 22_28, 22_29, 22_30, 22_31: TSOP2240, ShortCircuitRobotics:TSOP22XX
- removed C49, C51, C53, C55, C57, C59, C61, C63: 1µF, resistor:C1206
- removed C50, C52, C54, C56, C58, C60, C62, C64: 4.7µF, resistor:C1206
- removed IC4: 4051D, 40xx:SO16
- removed R49, R51, R53, R55, R57, R59, R61, R63: 100k, resistor:M1206
- removed R50, R52, R54, R56, R58, R60, R62, R64: 100, resistor:M1206
- moved JP4 316.9 mm to (-57.1, 17.1), turned to 180 degrees
- moved R78 301.0 mm to (-62.2, 8.89)
- moved TSOP_LED 299.3 mm to (-35.6, -12.7), turned to 180 degrees
- moved JP5 298.9 mm to (-37.5, -7.62), turned to 90 degrees
- moved R79 296.9 mm to (-34.3, -8.89), turned to 90 degrees
- moved R77 294.6 mm to (-56.5, 8.89), turned to 180 degrees
- moved JP3 273.1 mm to (-59.1, -7.62)
- moved R74 256.3 mm to (-19.7, -12.1), turned to 180 degrees
- moved R73 252.2 mm to (-14.0, -12.1), turned to 180 degrees
- moved R76 247.5 mm to (-24.1, -30.5), turned to 180 degrees
- moved R75 241.7 mm to (-29.8, -30.5)
- moved R70 237.2 mm to (-14.0, -8.26), turned to 180 degrees
- moved R69 230.0 mm to (-19.7, -8.26), turned to 180 degrees
- moved R72 229.7 mm to (-29.8, -26.0)
- moved JP2 225.6 mm to (-36.8, 26.7)
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Connections:
- removed net MUX_INH_3: IC4.6, IC5.11
- removed net N$49: 22_24.VCC, C50.1, R50.1
- removed net N$50: 22_24.OUT, R49.1
- removed net N$51: 22_25.VCC, C52.1, R52.1
- removed net N$52: 22_25.OUT, R51.1
- removed net N$53: 22_26.VCC, C54.1, R54.1
- removed net N$54: 22_26.OUT, R53.1
- removed net N$55: 22_27.VCC, C56.1, R56.1
- removed net N$56: 22_27.OUT, R55.1
- removed net N$57: 22_28.VCC, C58.1, R58.1
- removed net N$58: 22_28.OUT, R57.1
- removed net N$59: 22_29.VCC, C60.1, R60.1
- removed net N$60: 22_29.OUT, R59.1
- removed net N$61: 22_30.VCC, C62.1, R62.1
- removed net N$62: 22_30.OUT, R61.1
- removed net N$63: 22_31.VCC, C64.1, R64.1
- removed net N$64: 22_31.OUT, R63.1
- removed net TSOP24: C55.1, IC4.13, R55.2
- removed net TSOP25: C53.1, IC4.14, R53.2
- removed net TSOP26: C51.1, IC4.15, R51.2
- removed net TSOP27: C49.1, IC4.12, R49.2
- removed net TSOP28: C63.1, IC4.1, R63.2
- removed net TSOP29: C61.1, IC4.5, R61.2
- removed net TSOP30: C59.1, IC4.2, R59.2
- removed net TSOP31: C57.1, IC4.4, R57.2
- net GND: now also C66.2; no longer 22_24.GND, 22_25.GND, 22_26.GND, 22_27.GND, 22_28.GND, 22_29.GND, 22_30.GND, 22_31.GND, C49.2, C50.2, C51.2, C52.2, C53.2, C54.2, C55.2, C56.2, C57.2, C58.2, C59.2, C60.2, C61.2, C62.2, C63.2, C64.2, IC4.8
- net MUX_A: no longer IC4.11
- net MUX_B: no longer IC4.10
- net MUX_C: no longer IC4.9
- net MUX_OUT: no longer IC4.3
- net N$81: now also IC5.10
- net VCC: no longer C66.2, IC4.16
- net VEE: no longer IC4.7
- net VTSOP_A: no longer R50.2, R58.2
- net VTSOP_B: no longer R52.2, R60.2
- net VTSOP_C: no longer R54.2, R62.2
- net VTSOP_D: no longer R56.2, R64.2
Routing:
- net GND: track 0.00 -> 41.1 mm
- net N$11: track 0.00 -> 8.55 mm
- net N$13: track 0.00 -> 8.50 mm
- net N$9: track 0.00 -> 8.26 mm
- net N$6: track 0.00 -> 8.03 mm
- net N$47: track 0.00 -> 7.83 mm
- net N$8: track 0.00 -> 7.76 mm
- net N$3: track 0.00 -> 7.42 mm
- net N$1: track 0.00 -> 7.03 mm
- net N$17: track 0.00 -> 6.80 mm
- net N$15: track 0.00 -> 6.55 mm
- net N$14: track 0.00 -> 5.18 mm
- net N$12: track 0.00 -> 5.00 mm
- net N$7: track 0.00 -> 4.69 mm
- net N$2: track 0.00 -> 4.60 mm
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Other:
- board size 100 x 80 mm -> 201.2 x 155.2 mm

Commit message: TSOP: finished TSOP.sch and TSOP.brd 	TSOP data wires were connected with wrong TSOPS
Parts:
- moved U$1 25.8 mm to (-12.7, -27.3), flipped to the bottom, turned to 180 degrees
- moved R76 14.7 mm to (-22.9, -15.9), flipped to the bottom, turned to 0 degrees
- moved R75 14.6 mm to (-29.2, -15.9), flipped to the bottom, turned to 180 degrees
- moved R70 11.4 mm to (-10.2, -19.1), flipped to the bottom, turned to 0 degrees
- moved R69 11.3 mm to (-16.5, -19.1), flipped to the bottom
- moved R31 10.4 mm to (85.4, -28.4), turned to 180 degrees
- moved R32 10.3 mm to (81.6, -33.1), turned to 270 degrees
- moved C29 9.78 mm to (85.1, 3.10), turned to 180 degrees
- moved JP2 9.25 mm to (-27.9, 24.1), turned to 180 degrees
- moved R30 8.97 mm to (87.9, -1.52), turned to 270 degrees
- moved C45 8.82 mm to (-34.8, -40.7), turned to 90 degrees
- moved C43 8.26 mm to (-22.4, -40.1), turned to 90 degrees
- moved C27 7.81 mm to (90.2, 14.4), turned to 270 degrees
- moved R20 7.65 mm to (48.0, 74.1)
- moved U$2 7.65 mm to (-25.4, -27.3), flipped to the bottom, turned to 180 degrees
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Connections:
- removed net VEE: IC1.7, IC2.7, IC3.7
- net GND: now also IC1.7, IC2.7, IC3.7
- net TSOP0: now also C28.1, R13.2; no longer C6.1, R6.2
- net TSOP1: now also C1.1, R2.2; no longer C3.1, R4.2
- net TSOP10: now also C20.1, R21.2; no longer C18.1, R19.2
- net TSOP11: now also C22.1, R23.2; no longer C16.1, R17.2
- net TSOP12: now also C24.1, R25.2; no longer C31.1, R31.2
- net TSOP13: now also C26.1, R27.2; no longer C29.1, R29.2
- net TSOP14: now also C29.1, R29.2; no longer C26.1, R27.2
- net TSOP15: now also C31.1, R31.2; no longer C24.1, R25.2
- net TSOP16: now also C33.1, R33.2; no longer C39.1, R39.2
- net TSOP17: now also C35.1, R35.2; no longer C37.1, R37.2
- net TSOP18: now also C37.1, R37.2; no longer C35.1, R35.2
- net TSOP19: now also C39.1, R39.2; no longer C33.1, R33.2
- net TSOP2: now also C3.1, R4.2; no longer C1.1, R2.2
- net TSOP20: now also C41.1, R41.2; no longer C47.1, R47.2
- net TSOP21: now also C43.1, R43.2; no longer C45.1, R45.2
- net TSOP22: now also C45.1, R45.2; no longer C43.1, R43.2
- net TSOP23: now also C47.1, R47.2; no longer C41.1, R41.2
- net TSOP3: now also C6.1, R6.2; no longer C28.1, R13.2
- net TSOP4: now also C8.1, R8.2; no longer C14.1, R15.2
- net TSOP5: now also C10.1, R10.2; no longer C12.1, R12.2
- net TSOP6: now also C12.1, R12.2; no longer C10.1, R10.2
- net TSOP7: now also C14.1, R15.2; no longer C8.1, R8.2
- net TSOP8: now also C16.1, R17.2; no longer C22.1, R23.2
- net TSOP9: now also C18.1, R19.2; no longer C20.1, R21.2
Routing:
- net GND: track 41.1 -> 1321.9 mm, vias 0 -> 4
- net VTSOP_C: track 0.00 -> 510.9 mm, vias 0 -> 11
- net VTSOP_A: track 0.00 -> 467.2 mm, vias 0 -> 12
- net VTSOP_D: track 0.00 -> 463.0 mm, vias 0 -> 7
- net VTSOP_B: track 0.00 -> 460.4 mm, vias 0 -> 13
- net VCC: track 0.00 -> 445.4 mm, vias 0 -> 13
- net MUX_A: track 0.00 -> 350.0 mm, vias 0 -> 2
- net MUX_B: track 0.00 -> 339.2 mm, vias 0 -> 2
- net MUX_C: track 0.00 -> 331.0 mm, vias 0 -> 3
- net MUX_OUT: track 0.00 -> 324.0 mm, vias 0 -> 16
- net MUX_INH_1: track 0.00 -> 247.5 mm, vias 0 -> 7
- net TSOP7: track 2.74 -> 113.0 mm, vias 0 -> 4
- net TSOP15: track 0.00 -> 103.4 mm, vias 0 -> 4
- net RESET: track 0.00 -> 99.0 mm, vias 0 -> 7
- net TSOP0: track 2.79 -> 99.3 mm, vias 0 -> 4
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Other:
- outline, holes or cut-outs redrawn

Commit message: TSOP: cutting unneeded stuff off
Routing:
- net TSOP14: track 76.7 -> 81.6 mm
- net TSOP15: track 103.4 -> 106.3 mm
- net MUX_OUT: track 324.0 -> 326.7 mm
- net TSOP12: track 55.0 -> 52.8 mm
- net TSOP13: track 72.0 -> 72.8 mm
Other:
- outline, holes or cut-outs redrawn
