File: ec_motor_board.sch (EAGLE design)
At the start: 23 parts

Commit message: ec_motor_board: necessary pullups to 3.3v connected to hall sensors leiton.dru: added for drc with leiton values
Parts:
- added R10, R11, R12: (no value), resistor:R-EU_R1206
Connections:
- net N$19: now also R10.1
- net N$21: now also R11.2
- net N$23: now also R12.2
- net VCC: now also R10.2, R11.1, R12.1
Changed lines of the file:
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@@
 <part name="GND8" library="supply1" deviceset="GND" device=""/>
 <part name="C9" library="resistor" deviceset="C-EU" device="C1206" value="100nF"/>
+<part name="R10" library="resistor" deviceset="R-EU_" device="R1206"/>
+<part name="R11" library="resistor" deviceset="R-EU_" device="R1206"/>
+<part name="P+5" library="supply1" deviceset="VCC" device=""/>
+<part name="P+6" library="supply1" deviceset="VCC" device=""/>
+<part name="R12" library="resistor" deviceset="R-EU_" device="R1206"/>
+<part name="P+7" library="supply1" deviceset="VCC" device=""/>
 </parts>
 <sheets>
@@
 <instance part="GND8" gate="1" x="48.26" y="-7.62" rot="R270"/>
 <instance part="C9" gate="G$1" x="-33.02" y="45.72" rot="R270"/>
+<instance part="R10" gate="G$1" x="17.78" y="20.32" rot="R90"/>
+<instance part="R11" gate="G$1" x="22.86" y="10.16" rot="R180"/>
+<instance part="P+5" gate="VCC" x="17.78" y="30.48"/>
+<instance part="P+6" gate="VCC" x="33.02" y="10.16" rot="R270"/>
+<instance part="R12" gate="G$1" x="33.02" y="-7.62" rot="R180"/>
+<instance part="P+7" gate="VCC" x="43.18" y="-7.62" rot="R270"/>
 </instances>
 <busses>
@@
 <segment>
 <pinref part="ROW1" gate="A" pin="3"/>
-<wire x1="60.96" y1="10.16" x2="33.02" y2="10.16" width="0.1524" layer="91"/>
-<wire x1="33.02" y1="10.16" x2="33.02" y2="17.78" width="0.1524" layer="91"/>
+<wire x1="60.96" y1="10.16" x2="40.64" y2="10.16" width="0.1524" layer="91"/>
+<wire x1="40.64" y1="10.16" x2="40.64" y2="17.78" width="0.1524" layer="91"/>
 <pinref part="U$1" gate="G$1" pin="OUT_1"/>
-<wire x1="33.02" y1="17.78" x2="15.24" y2="17.78" width="0.1524" layer="91"/>
+<wire x1="40.64" y1="17.78" x2="15.24" y2="17.78" width="0.1524" layer="91"/>
 </segment>
 </net>
@@
 <segment>
 <pinref part="U$1" gate="G$1" pin="H_1"/>
-<wire x1="15.24" y1="15.24" x2="30.48" y2="15.24" width="0.1524" layer="91"/>
-<wire x1="30.48" y1="15.24" x2="30.48" y2="7.62" width="0.1524" layer="91"/>
+<wire x1="15.24" y1="15.24" x2="17.78" y2="15.24" width="0.1524" layer="91"/>
+<wire x1="17.78" y1="15.24" x2="38.1" y2="15.24" width="0.1524" layer="91"/>
+<wire x1="38.1" y1="15.24" x2="38.1" y2="7.62" width="0.1524" layer="91"/>
 <pinref part="ROW1" gate="A" pin="4"/>
-<wire x1="30.48" y1="7.62" x2="60.96" y2="7.62" width="0.1524" layer="91"/>
+<wire x1="38.1" y1="7.62" x2="60.96" y2="7.62" width="0.1524" layer="91"/>
+<pinref part="R10" gate="G$1" pin="1"/>
+<junction x="17.78" y="15.24"/>
 </segment>
 </net>
@@
 <segment>
 <pinref part="U$1" gate="G$1" pin="H_2"/>
-<wire x1="15.24" y1="5.08" x2="25.4" y2="5.08" width="0.1524" layer="91"/>
+<wire x1="15.24" y1="5.08" x2="17.78" y2="5.08" width="0.1524" layer="91"/>
+<wire x1="17.78" y1="5.08" x2="25.4" y2="5.08" width="0.1524" layer="91"/>
 <wire x1="25.4" y1="5.08" x2="25.4" y2="2.54" width="0.1524" layer="91"/>
 <pinref part="ROW1" gate="A" pin="6"/>
 <wire x1="25.4" y1="2.54" x2="60.96" y2="2.54" width="0.1524" layer="91"/>
+<pinref part="R11" gate="G$1" pin="2"/>
+<wire x1="17.78" y1="10.16" x2="17.78" y2="5.08" width="0.1524" layer="91"/>
+<junction x="17.78" y="5.08"/>
 </segment>
 </net>
@@
 <segment>
 <pinref part="U$1" gate="G$1" pin="H_3"/>
-<wire x1="15.24" y1="-5.08" x2="27.94" y2="-5.08" width="0.1524" layer="91"/>
+<wire x1="15.24" y1="-5.08" x2="25.4" y2="-5.08" width="0.1524" layer="91"/>
+<wire x1="25.4" y1="-5.08" x2="27.94" y2="-5.08" width="0.1524" layer="91"/>
 <wire x1="27.94" y1="-5.08" x2="27.94" y2="-2.54" width="0.1524" layer="91"/>
 <wire x1="27.94" y1="-2.54" x2="60.96" y2="-2.54" width="0.1524" layer="91"/>
 <pinref part="ROW1" gate="A" pin="8"/>
+<pinref part="R12" gate="G$1" pin="2"/>
+<wire x1="27.94" y1="-7.62" x2="25.4" y2="-7.62" width="0.1524" layer="91"/>
+<wire x1="25.4" y1="-7.62" x2="25.4" y2="-5.08" width="0.1524" layer="91"/>
+<junction x="25.4" y="-5.08"/>
 </segment>
 </net>
@@
 <pinref part="P+3" gate="VCC" pin="VCC"/>
 </segment>
-</net>
+<segment>
+<pinref part="R10" gate="G$1" pin="2"/>
+<pinref part="P+5" gate="VCC" pin="VCC"/>
+<wire x1="17.78" y1="27.94" x2="17.78" y2="25.4" width="0.1524" layer="91"/>
+</segment>
+<segment>
+<pinref part="R11" gate="G$1" pin="1"/>
+<pinref part="P+6" gate="VCC" pin="VCC"/>
+<wire x1="30.48" y1="10.16" x2="27.94" y2="10.16" width="0.1524" layer="91"/>
+</segment>
+<segment>
+<pinref part="R12" gate="G$1" pin="1"/>
+<pinref part="P+7" gate="VCC" pin="VCC"/>
+<wire x1="40.64" y1="-7.62" x2="38.1" y2="-7.62" width="0.1524" layer="91"/>
+</segment>
+</net>

Commit message: ec_motor_board: added an 0 ohm resistor which can connect vref to vcc to disable power regulation
Parts:
- added R13: 0, resistor:R-EU_R1206
Connections:
- net N$14: now also R13.2
- net VCC: now also R13.1
Other:
- moved on the sheet: R7
Changed lines of the file:
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@@
 <part name="R12" library="resistor" deviceset="R-EU_" device="R1206"/>
 <part name="P+7" library="supply1" deviceset="VCC" device=""/>
+<part name="R13" library="resistor" deviceset="R-EU_" device="R1206" value="0"/>
+<part name="P+8" library="supply1" deviceset="VCC" device=""/>
 </parts>
 <sheets>
@@
 <instance part="D2" gate="G$1" x="-27.94" y="30.48" rot="R180"/>
 <instance part="R6" gate="G$1" x="-55.88" y="-12.7" rot="R90"/>
-<instance part="R7" gate="G$1" x="-68.58" y="-7.62"/>
+<instance part="R7" gate="G$1" x="-63.5" y="-7.62"/>
 <instance part="R8" gate="G$1" x="33.02" y="-12.7"/>
 <instance part="R9" gate="G$1" x="33.02" y="-10.16"/>
@@
 <instance part="R12" gate="G$1" x="33.02" y="-7.62" rot="R180"/>
 <instance part="P+7" gate="VCC" x="43.18" y="-7.62" rot="R270"/>
+<instance part="R13" gate="G$1" x="-73.66" y="-12.7" rot="R90"/>
+<instance part="P+8" gate="VCC" x="-73.66" y="-22.86" rot="R180"/>
 </instances>
 <busses>
@@
 <pinref part="R6" gate="G$1" pin="2"/>
 <junction x="-55.88" y="-7.62"/>
-<wire x1="-55.88" y1="-7.62" x2="-63.5" y2="-7.62" width="0.1524" layer="91"/>
+<wire x1="-55.88" y1="-7.62" x2="-58.42" y2="-7.62" width="0.1524" layer="91"/>
 <pinref part="R7" gate="G$1" pin="2"/>
 </segment>
@@
 <segment>
 <pinref part="R7" gate="G$1" pin="1"/>
+<wire x1="-68.58" y1="-7.62" x2="-73.66" y2="-7.62" width="0.1524" layer="91"/>
 <wire x1="-73.66" y1="-7.62" x2="-76.2" y2="-7.62" width="0.1524" layer="91"/>
 <wire x1="-76.2" y1="-7.62" x2="-76.2" y2="-5.08" width="0.1524" layer="91"/>
 <pinref part="ROW2" gate="A" pin="8"/>
 <wire x1="-76.2" y1="-5.08" x2="-96.52" y2="-5.08" width="0.1524" layer="91"/>
+<pinref part="R13" gate="G$1" pin="2"/>
+<junction x="-73.66" y="-7.62"/>
 </segment>
 </net>
@@
 <wire x1="40.64" y1="-7.62" x2="38.1" y2="-7.62" width="0.1524" layer="91"/>
 </segment>
-</net>
+<segment>
+<pinref part="R13" gate="G$1" pin="1"/>
+<pinref part="P+8" gate="VCC" pin="VCC"/>
+<wire x1="-73.66" y1="-20.32" x2="-73.66" y2="-17.78" width="0.1524" layer="91"/>
+</segment>
+</net>

Commit message: MainBoard: replaced old version of Kevin with new version of Christoph 		moved Light Barrier connections to bottom layer
Changed lines of the file:
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@@
 <wire x1="-43.18" y1="45.72" x2="-38.1" y2="45.72" width="0.1524" layer="91"/>
 <junction x="-43.18" y="38.1"/>
+<junction x="-43.18" y="30.48"/>
 </segment>
 </net>
