File: main_board.brd (EAGLE design)
At the start: 201.2 x 155.4 mm, 206 parts, among them IC10 MEGA48/88/168-PU, IC11 MEGA48/88/168-PU, IC2 LM567N, IC3 74AC11000D, IC4 4050D, IC5 ATMEGA644-20PU, IC6 4051D, IC7 AD8655R, IC8 4051D, IC9 TINY24/44/84-SSU, J1 22-27-2041-04, K2 4052, Q2 MOSFET-NCHANNELSMD, U1 XC9572VQ44

Commit message: Main: Changed MUX-EN to MUX-INH. This pin should have been called INHIBIT  in the first place because it is LOW ACTIVE!!!!!
Connections:
- net MUX1-EN renamed MUX1-INH
- new net MUX2-INH: IC8.6
- net MUX2-EN: no longer IC8.6
Routing:
- net MUX2-EN: track 73.1 -> 71.1 mm
Changed lines of the file:
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@@
 <via x="14.732" y="80.1878" extent="1-16" drill="0.6"/>
 </signal>
-<signal name="MUX1-EN">
+<signal name="MUX1-INH">
 <contactref element="IC6" pad="6"/>
 <contactref element="IC11" pad="12"/>
@@
 </signal>
 <signal name="MUX2-EN">
-<contactref element="IC8" pad="6"/>
 <contactref element="IC11" pad="13"/>
 <wire x1="41.91" y1="28.1178" x2="39.37" y2="28.1178" width="0.4064" layer="16"/>
@@
 <wire x1="38.1" y1="26.8478" x2="32.385" y2="26.8478" width="0.4064" layer="16"/>
 <wire x1="30.48" y1="28.7528" x2="30.48" y2="66.2178" width="0.4064" layer="1"/>
-<wire x1="29.7434" y1="86.5378" x2="31.75" y2="86.5378" width="0.4064" layer="1"/>
 <via x="31.75" y="86.5378" extent="1-16" drill="0.6"/>
 <wire x1="31.75" y1="86.5378" x2="30.48" y2="85.2678" width="0.4064" layer="16"/>
@@
 <wire x1="-7.62" y1="-6.985" x2="-9.525" y2="-6.985" width="0.4064" layer="16"/>
 </signal>
+<signal name="MUX2-INH">
+<contactref element="IC8" pad="6"/>
+</signal>
 </signals>

Commit message: MainBoard: Fixed Motor Controller Connections Moved them to the lower layer.
Routing:
- net RESET_MOTOR: track 42.0 -> 41.7 mm, vias 3 -> 4
- net MC_IN_B: vias 3 -> 4
Changed lines of the file:
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@@
 <?xml version="1.0" encoding="utf-8"?>
 <!DOCTYPE eagle SYSTEM "eagle.dtd">
-<eagle version="6.2">
+<eagle version="6.3">
 <drawing>
 <settings>
@@
 </class>
 </classes>
-<designrules>
+<designrules name="default">
 <description language="de">&lt;b&gt;EAGLE Design Rules&lt;/b&gt;
 &lt;p&gt;
@@
 <wire x1="16.51" y1="63.6778" x2="16.51" y2="63.0428" width="0.4064" layer="16"/>
 <via x="16.51" y="63.0428" extent="1-16" drill="0.6"/>
-<wire x1="-4.445" y1="38.9128" x2="0.635" y2="38.9128" width="0.4064" layer="1"/>
-<wire x1="0.635" y1="38.9128" x2="1.905" y2="40.8178" width="0.4064" layer="1"/>
-<wire x1="1.905" y1="40.8178" x2="3.175" y2="40.8178" width="0.4064" layer="1"/>
+<wire x1="0.8128" y1="40.8178" x2="3.175" y2="40.8178" width="0.4064" layer="1"/>
 <wire x1="3.175" y1="40.8178" x2="4.445" y2="42.0878" width="0.4064" layer="1"/>
 <via x="4.445" y="42.0878" extent="1-16" drill="0.6"/>
@@
 <wire x1="15.875" y1="55.245" x2="14.605" y2="55.245" width="0.4064" layer="1"/>
 <wire x1="14.605" y1="55.245" x2="12.8778" y2="53.5178" width="0.4064" layer="1"/>
+<wire x1="-4.445" y1="38.9128" x2="-1.0922" y2="38.9128" width="0.4064" layer="16"/>
+<wire x1="-1.0922" y1="38.9128" x2="-0.635" y2="39.37" width="0.4064" layer="16"/>
+<via x="-0.635" y="39.37" extent="1-16" drill="0.6"/>
+<wire x1="-0.635" y1="39.37" x2="0.8128" y2="40.8178" width="0.4064" layer="1"/>
 </signal>
 <signal name="N$50">
@@
 <wire x1="-8.255" y1="-29.0322" x2="-3.81" y2="-24.5872" width="0.4064" layer="16"/>
 <wire x1="-3.81" y1="-24.5872" x2="-3.81" y2="-6.1722" width="0.4064" layer="16"/>
-<wire x1="-7.62" y1="7.1628" x2="-7.62" y2="-2.3622" width="0.4064" layer="1"/>
 <via x="-7.62" y="-2.3622" extent="1-16" drill="0.6"/>
+<wire x1="-7.62" y1="6.985" x2="-7.62" y2="-2.3622" width="0.4064" layer="1"/>
 <wire x1="-7.62" y1="-2.3622" x2="-3.81" y2="-6.1722" width="0.4064" layer="16"/>
 <contactref element="IC10" pad="13"/>
-<wire x1="-7.62" y1="7.1628" x2="-6.35" y2="8.4328" width="0.4064" layer="1"/>
-<wire x1="-6.35" y1="8.4328" x2="-4.445" y2="8.4328" width="0.4064" layer="1"/>
+<wire x1="-4.445" y1="8.4328" x2="-6.35" y2="8.4328" width="0.4064" layer="16"/>
+<wire x1="-6.35" y1="8.4328" x2="-7.62" y2="7.1628" width="0.4064" layer="16"/>
+<via x="-7.62" y="7.1628" extent="1-16" drill="0.6"/>
+<wire x1="-7.62" y1="7.1628" x2="-7.62" y2="6.985" width="0.4064" layer="1"/>
 </signal>
 <signal name="MC_DIAG_A">

Commit message: MainBoard: replaced old version of Kevin with new version of Christoph 		moved Light Barrier connections to bottom layer
Parts:
- JP4: device pinhead:1X02 -> pinhead:1X01
- moved JP4 1.27 mm to (14.6, -15.9)
- flipped LB_LED to the bottom
Connections:
- removed net N$110: IC5.34, JP4.2
- net KICKER_ON: now also IC5.34; no longer IC5.12
Routing:
- net KICKER_ON: track 51.9 -> 73.7 mm
- net N$7: track 5.94 -> 11.9 mm, vias 0 -> 1
- net N$110: track 4.27 -> 0.00 mm
- net N$6: track 3.17 -> 7.14 mm, vias 0 -> 1
- net MC_EN: track 123.0 -> 125.2 mm
- net GND: track 2043.5 -> 2044.9 mm, vias 52 -> 53
- net MISO: track 278.1 -> 278.6 mm, vias 5 -> 7
- net RESET_MOTOR: track 41.7 -> 41.4 mm, vias 4 -> 2
- net N$10: vias 1 -> 0

Commit message: ShortCircuitLbr: 74HC00D in SO14 Package added MainBoard: replaced wrong nand-gate package (for DIAG Pins) with 74HC00D SO14
Parts:
- removed IC3: 74AC11000D, 74ac-logic:SO16
- added U$10: 74HC00, ShortCircuitRobotics:SO14
Connections:
- net GND: now also U$10.7; no longer IC3.4, IC3.5
- net MA_DIAG: now also U$10.3; no longer IC3.2
- net MA_DIAG_A: now also U$10.2; no longer IC3.1
- net MA_DIAG_B: now also U$10.1; no longer IC3.16
- net MB_DIAG: now also U$10.6; no longer IC3.3
- net MB_DIAG_A: now also U$10.5; no longer IC3.15
- net MB_DIAG_B: now also U$10.4; no longer IC3.14
- net MC_DIAG: now also U$10.8; no longer IC3.6
- net MC_DIAG_A: now also U$10.10; no longer IC3.11
- net MC_DIAG_B: now also U$10.9; no longer IC3.10
- net MD_DIAG: now also U$10.11; no longer IC3.7
- net MD_DIAG_A: now also U$10.13; no longer IC3.9
- net MD_DIAG_B: now also U$10.12; no longer IC3.8
- net VCC: now also U$10.14; no longer IC3.12, IC3.13
Routing:
- net VCC: track 685.9 -> 699.1 mm, vias 26 -> 28
- net GND: track 2044.9 -> 2033.2 mm
- net MA_DIAG_B: track 44.5 -> 56.0 mm
- net MC_DIAG_A: track 90.4 -> 79.9 mm
- net MA_DIAG_A: track 51.3 -> 59.3 mm
- net MC_DIAG_B: track 81.5 -> 75.7 mm
- net MD_DIAG: track 33.7 -> 37.3 mm
- net MD_DIAG_B: track 57.2 -> 60.9 mm
- net MD_DIAG_A: track 60.8 -> 59.1 mm
- net MA_IN_B: track 84.0 -> 83.2 mm
- net MB_DIAG_A: track 13.0 -> 13.7 mm
- net N$87: track 30.9 -> 31.6 mm
