File: main_board.sch (EAGLE design)
At the start: 206 parts, among them IC10 MEGA48/88/168-PU, IC11 MEGA48/88/168-PU, IC2 LM567N, IC3 74AC11000D, IC4 4050D, IC5 ATMEGA644-20PU, IC6 4051D, IC7 AD8655R, IC8 4051D, IC9 TINY24/44/84-SSU, J1 22-27-2041-04, K2 4052, Q2 MOSFET-NCHANNELSMD, U1 XC9572VQ44

Commit message: Main: Changed MUX-EN to MUX-INH. This pin should have been called INHIBIT  in the first place because it is LOW ACTIVE!!!!!
Connections:
- net MUX1-EN renamed MUX1-INH
- new net MUX2-INH: IC8A.INH
- net MUX2-EN: no longer IC8A.INH
Changed lines of the file:
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@@
 </segment>
 </net>
-<net name="MUX1-EN" class="0">
+<net name="MUX1-INH" class="0">
 <segment>
 <wire x1="144.78" y1="25.4" x2="149.86" y2="25.4" width="0.1524" layer="91"/>
@@
 <label x="149.86" y="22.86" size="1.27" layer="95" xref="yes"/>
 <pinref part="IC11" gate="1" pin="PD7(AIN1/PCINT23)"/>
-</segment>
-<segment>
-<pinref part="IC8" gate="A" pin="INH"/>
-<wire x1="50.8" y1="-132.08" x2="27.94" y2="-132.08" width="0.1524" layer="91"/>
-<label x="27.94" y="-132.08" size="1.016" layer="95" rot="MR0" xref="yes"/>
 </segment>
 </net>
@@
 </segment>
 </net>
+<net name="MUX2-INH" class="0">
+<segment>
+<pinref part="IC8" gate="A" pin="INH"/>
+<wire x1="50.8" y1="-132.08" x2="27.94" y2="-132.08" width="0.1524" layer="91"/>
+<label x="27.94" y="-132.08" size="1.016" layer="95" rot="MR0" xref="yes"/>
+</segment>
+</net>

Commit message: MainBoard: replaced old version of Kevin with new version of Christoph 		moved Light Barrier connections to bottom layer
Parts:
- JP4: device pinhead:PINHD-1X2 -> pinhead:PINHD-1X1
Connections:
- removed net N$110: IC5.PCINT6/ADC6_PA6, JP4.2
- net KICKER_ON: now also IC5.PCINT6/ADC6_PA6; no longer IC5.XTAL2
Changed lines of the file:
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@@
 <part name="P+44" library="supply1" deviceset="VCC" device=""/>
 <part name="GND76" library="supply1" deviceset="GND" device=""/>
-<part name="JP4" library="pinhead" deviceset="PINHD-1X2" device=""/>
+<part name="JP4" library="pinhead" deviceset="PINHD-1X1" device=""/>
 <part name="GND_A" library="pinhead" deviceset="PINHD-1X1" device=""/>
 <part name="GND_B" library="pinhead" deviceset="PINHD-1X1" device=""/>
@@
 <instance part="P+44" gate="VCC" x="307.34" y="66.04" rot="R90"/>
 <instance part="GND76" gate="1" x="314.96" y="60.96" rot="R270"/>
-<instance part="JP4" gate="G$1" x="373.38" y="218.44"/>
+<instance part="JP4" gate="G$1" x="373.38" y="220.98"/>
 <instance part="GND_A" gate="G$1" x="281.94" y="81.28"/>
 <instance part="GND_B" gate="G$1" x="281.94" y="73.66"/>
@@
 </segment>
 <segment>
-<pinref part="IC5" gate="G$1" pin="XTAL2"/>
-<wire x1="279.4" y1="205.74" x2="266.7" y2="205.74" width="0.1524" layer="91"/>
-<label x="266.7" y="205.74" size="1.778" layer="95" rot="MR0" xref="yes"/>
+<pinref part="IC5" gate="G$1" pin="PCINT6/ADC6_PA6"/>
+<wire x1="340.36" y1="218.44" x2="345.44" y2="218.44" width="0.1524" layer="91"/>
+<label x="345.44" y="218.44" size="1.27" layer="95" xref="yes"/>
 </segment>
 </net>
@@
 </segment>
 </net>
-<net name="N$110" class="0">
-<segment>
-<pinref part="IC5" gate="G$1" pin="PCINT6/ADC6_PA6"/>
-<wire x1="340.36" y1="218.44" x2="370.84" y2="218.44" width="0.1524" layer="91"/>
-<pinref part="JP4" gate="G$1" pin="2"/>
-</segment>
-</net>

Commit message: ShortCircuitLbr: 74HC00D in SO14 Package added MainBoard: replaced wrong nand-gate package (for DIAG Pins) with 74HC00D SO14
Parts:
- removed IC3: 74AC11000D, 74ac-logic:74AC11000D
- added U$10: 74HC00, ShortCircuitRobotics:74HC00
Connections:
- net GND: now also U$10G$5.GND; no longer IC3P.GND@1, IC3P.GND@2
- net MA_DIAG: now also U$10G$1.O; no longer IC3A.O
- net MA_DIAG_A: now also U$10G$1.I1; no longer IC3A.I0
- net MA_DIAG_B: now also U$10G$1.I0; no longer IC3A.I1
- net MB_DIAG: now also U$10G$2.O; no longer IC3B.O
- net MB_DIAG_A: now also U$10G$2.I1; no longer IC3B.I0
- net MB_DIAG_B: now also U$10G$2.I0; no longer IC3B.I1
- net MC_DIAG: now also U$10G$3.O; no longer IC3C.O
- net MC_DIAG_A: now also U$10G$3.I1; no longer IC3C.I0
- net MC_DIAG_B: now also U$10G$3.I0; no longer IC3C.I1
- net MD_DIAG: now also U$10G$4.O; no longer IC3D.O
- net MD_DIAG_A: now also U$10G$4.I1; no longer IC3D.I0
- net MD_DIAG_B: now also U$10G$4.I0; no longer IC3D.I1
- net VCC: now also U$10G$5.PWR; no longer IC3P.VCC@1, IC3P.VCC@2
Changed lines of the file:
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@@
 <part name="P+17" library="supply1" deviceset="VCC" device=""/>
 <part name="GND64" library="supply1" deviceset="GND" device=""/>
-<part name="IC3" library="74ac-logic" deviceset="74AC11000" device="D"/>
 <part name="GND17" library="supply1" deviceset="GND" device=""/>
 <part name="P+37" library="supply1" deviceset="VCC" device=""/>
@@
 <part name="GND_E" library="pinhead" deviceset="PINHD-1X1" device=""/>
 <part name="GND77" library="supply1" deviceset="GND" device=""/>
+<part name="U$10" library="ShortCircuitRobotics" deviceset="74HC00" device=""/>
 </parts>
 <sheets>
@@
 <instance part="P+17" gate="VCC" x="652.78" y="-121.92" rot="MR270"/>
 <instance part="GND64" gate="1" x="647.7" y="-137.16" rot="R270"/>
-<instance part="IC3" gate="A" x="411.48" y="-50.8" rot="MR0"/>
-<instance part="IC3" gate="B" x="411.48" y="-160.02" rot="MR0"/>
-<instance part="IC3" gate="C" x="530.86" y="-53.34" rot="MR0"/>
-<instance part="IC3" gate="D" x="530.86" y="-162.56" rot="MR0"/>
-<instance part="IC3" gate="P" x="513.08" y="-251.46" rot="R270"/>
-<instance part="GND17" gate="1" x="495.3" y="-251.46" rot="R270"/>
-<instance part="P+37" gate="VCC" x="530.86" y="-251.46" rot="R270"/>
+<instance part="GND17" gate="1" x="502.92" y="-228.6" rot="R270"/>
+<instance part="P+37" gate="VCC" x="502.92" y="-233.68" rot="R90"/>
 <instance part="IC11" gate="1" x="114.3" y="35.56"/>
 <instance part="GND3" gate="1" x="68.58" y="7.62" rot="R270"/>
@@
 <instance part="GND_E" gate="G$1" x="281.94" y="50.8"/>
 <instance part="GND77" gate="1" x="261.62" y="66.04" rot="R270"/>
+<instance part="U$10" gate="G$1" x="411.48" y="-50.8" rot="R180"/>
+<instance part="U$10" gate="G$2" x="414.02" y="-160.02" rot="R180"/>
+<instance part="U$10" gate="G$3" x="530.86" y="-53.34" rot="R180"/>
+<instance part="U$10" gate="G$4" x="530.86" y="-162.56" rot="R180"/>
+<instance part="U$10" gate="G$5" x="513.08" y="-231.14" rot="R180"/>
 </instances>
 <busses>
@@
 </segment>
 <segment>
-<pinref part="IC3" gate="P" pin="GND@2"/>
-<pinref part="GND17" gate="1" pin="GND"/>
-<wire x1="497.84" y1="-251.46" x2="500.38" y2="-251.46" width="0.1524" layer="91"/>
-<wire x1="505.46" y1="-251.46" x2="500.38" y2="-251.46" width="0.1524" layer="91"/>
-<wire x1="500.38" y1="-251.46" x2="500.38" y2="-248.92" width="0.1524" layer="91"/>
-<pinref part="IC3" gate="P" pin="GND@1"/>
-<wire x1="500.38" y1="-248.92" x2="505.46" y2="-248.92" width="0.1524" layer="91"/>
-</segment>
-<segment>
 <pinref part="IC11" gate="1" pin="AGND"/>
 <pinref part="GND2" gate="1" pin="GND"/>
@@
 <junction x="271.78" y="58.42"/>
 </segment>
+<segment>
+<pinref part="U$10" gate="G$5" pin="GND"/>
+<pinref part="GND17" gate="1" pin="GND"/>
+<wire x1="505.46" y1="-228.6" x2="508" y2="-228.6" width="0.1524" layer="91"/>
+</segment>
 </net>
 <net name="MOSI" class="0">
@@
 </segment>
 <segment>
-<pinref part="IC3" gate="P" pin="VCC@2"/>
-<pinref part="P+37" gate="VCC" pin="VCC"/>
-<wire x1="528.32" y1="-251.46" x2="523.24" y2="-251.46" width="0.1524" layer="91"/>
-<pinref part="IC3" gate="P" pin="VCC@1"/>
-<wire x1="523.24" y1="-251.46" x2="520.7" y2="-251.46" width="0.1524" layer="91"/>
-<wire x1="520.7" y1="-248.92" x2="523.24" y2="-248.92" width="0.1524" layer="91"/>
-<wire x1="523.24" y1="-248.92" x2="523.24" y2="-251.46" width="0.1524" layer="91"/>
-</segment>
-<segment>
 <pinref part="IC11" gate="1" pin="AREF"/>
 <pinref part="P+4" gate="VCC" pin="VCC"/>
@@
 <pinref part="P+44" gate="VCC" pin="VCC"/>
 </segment>
+<segment>
+<pinref part="U$10" gate="G$5" pin="PWR"/>
+<pinref part="P+37" gate="VCC" pin="VCC"/>
+<wire x1="505.46" y1="-233.68" x2="508" y2="-233.68" width="0.1524" layer="91"/>
+</segment>
 </net>
 <net name="TSOP0" class="0">
@@
 <pinref part="U$4" gate="G$1" pin="DIAG_A/-"/>
 <wire x1="424.18" y1="-48.26" x2="419.1" y2="-48.26" width="0.1524" layer="91"/>
-<pinref part="IC3" gate="A" pin="I0"/>
+<pinref part="U$10" gate="G$1" pin="I1"/>
 </segment>
 </net>
@@
 <pinref part="U$4" gate="G$1" pin="DIAG_B/-"/>
 <wire x1="424.18" y1="-53.34" x2="419.1" y2="-53.34" width="0.1524" layer="91"/>
-<pinref part="IC3" gate="A" pin="I1"/>
+<pinref part="U$10" gate="G$1" pin="I0"/>
 </segment>
 </net>
@@
 <segment>
 <pinref part="U$6" gate="G$1" pin="DIAG_A/-"/>
-<wire x1="424.18" y1="-157.48" x2="419.1" y2="-157.48" width="0.1524" layer="91"/>
-<pinref part="IC3" gate="B" pin="I0"/>
+<wire x1="424.18" y1="-157.48" x2="421.64" y2="-157.48" width="0.1524" layer="91"/>
+<pinref part="U$10" gate="G$2" pin="I1"/>
 </segment>
 </net>
@@
 <segment>
 <pinref part="U$6" gate="G$1" pin="DIAG_B/-"/>
-<wire x1="424.18" y1="-162.56" x2="419.1" y2="-162.56" width="0.1524" layer="91"/>
-<pinref part="IC3" gate="B" pin="I1"/>
+<wire x1="424.18" y1="-162.56" x2="421.64" y2="-162.56" width="0.1524" layer="91"/>
+<pinref part="U$10" gate="G$2" pin="I0"/>
 </segment>
 </net>
@@
 <pinref part="U$5" gate="G$1" pin="DIAG_A/-"/>
 <wire x1="543.56" y1="-50.8" x2="538.48" y2="-50.8" width="0.1524" layer="91"/>
-<pinref part="IC3" gate="C" pin="I0"/>
+<pinref part="U$10" gate="G$3" pin="I1"/>
+<junction x="538.48" y="-50.8"/>
 </segment>
 </net>
@@
 <pinref part="U$5" gate="G$1" pin="DIAG_B/-"/>
 <wire x1="543.56" y1="-55.88" x2="538.48" y2="-55.88" width="0.1524" layer="91"/>
-<pinref part="IC3" gate="C" pin="I1"/>
+<pinref part="U$10" gate="G$3" pin="I0"/>
+<junction x="538.48" y="-55.88"/>
 </segment>
 </net>
@@
 <pinref part="U$7" gate="G$1" pin="DIAG_A/-"/>
 <wire x1="543.56" y1="-160.02" x2="538.48" y2="-160.02" width="0.1524" layer="91"/>
-<pinref part="IC3" gate="D" pin="I0"/>
+<pinref part="U$10" gate="G$4" pin="I1"/>
 </segment>
 </net>
@@
 <pinref part="U$7" gate="G$1" pin="DIAG_B/-"/>
 <wire x1="543.56" y1="-165.1" x2="538.48" y2="-165.1" width="0.1524" layer="91"/>
-<pinref part="IC3" gate="D" pin="I1"/>
+<pinref part="U$10" gate="G$4" pin="I0"/>
 </segment>
 </net>
@@
 <net name="MB_DIAG" class="0">
 <segment>
-<wire x1="403.86" y1="-160.02" x2="401.32" y2="-160.02" width="0.1524" layer="91"/>
+<wire x1="406.4" y1="-160.02" x2="401.32" y2="-160.02" width="0.1524" layer="91"/>
 <label x="401.32" y="-160.02" size="1.27" layer="95" rot="MR0" xref="yes"/>
-<pinref part="IC3" gate="B" pin="O"/>
+<pinref part="U$10" gate="G$2" pin="O"/>
 </segment>
 </net>
@@
 <wire x1="403.86" y1="-50.8" x2="401.32" y2="-50.8" width="0.1524" layer="91"/>
 <label x="401.32" y="-50.8" size="1.27" layer="95" rot="MR0" xref="yes"/>
-<pinref part="IC3" gate="A" pin="O"/>
+<pinref part="U$10" gate="G$1" pin="O"/>
 </segment>
 </net>
@@
 <wire x1="523.24" y1="-53.34" x2="520.7" y2="-53.34" width="0.1524" layer="91"/>
 <label x="520.7" y="-53.34" size="1.27" layer="95" rot="MR0" xref="yes"/>
-<pinref part="IC3" gate="C" pin="O"/>
+<pinref part="U$10" gate="G$3" pin="O"/>
+<junction x="523.24" y="-53.34"/>
 </segment>
 </net>
@@
 <wire x1="523.24" y1="-162.56" x2="520.7" y2="-162.56" width="0.1524" layer="91"/>
 <label x="520.7" y="-162.56" size="1.27" layer="95" rot="MR0" xref="yes"/>
-<pinref part="IC3" gate="D" pin="O"/>
+<pinref part="U$10" gate="G$4" pin="O"/>
 </segment>
 <segment>
